File: RELAY_MODULE_1_REV1.kicad_sch (KiCad schematic)
At the start: 54 parts, among them K1 SANYOU_SRD_Form_C, K2 SANYOU_SRD_Form_C, K3 SANYOU_SRD_Form_C, K4 SANYOU_SRD_Form_C, K5 SANYOU_SRD_Form_C, K6 SANYOU_SRD_Form_C, Q1 PN2222A, Q2 PN2222A, Q3 PN2222A, Q4 PN2222A, Q5 PN2222A, Q6 PN2222A

Commit message: BUGFIX: The Diagram error in to relay module was fixed.
The routing error in the relay diagram was fixed, also, a prototype of the relay circuit was build and the functionality was validated satisfactorily
Connections:
- net K2_COM: now reaches K2.1
- net K2_N_O: now reaches K2.3
- net K2_N_C: now reaches K2.4
- net K5_COM: now reaches K5.1
- net K5_N_O: now reaches K5.3
- net K5_N_C: now reaches K5.4
- net K6_COM: now reaches K6.1
- net K6_N_O: now reaches K6.3
- net K6_N_C: now reaches K6.4
- net K3_COM: now reaches K3.1
- net K3_N_O: now reaches K3.3
- net K3_N_C: now reaches K3.4
- net K4_COM: now reaches K4.1
- net K4_N_O: now reaches K4.3
- net K4_N_C: now reaches K4.4
- net K1_COM: now reaches K1.1
- net K1_N_O: now reaches K1.3
- net K1_N_C: now reaches K1.4
Other:
- moved on the sheet: D4, D5, D6, K4, K5, K6, O4, O5, O6, Q4, Q5, Q6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

Commit message: PCB REV 001 design
The design of the first revition of the PCB is complete.
Parts:
- removed R1, R16, R26, R6: 330, Resistor_THT:R_Axial_DIN0207_L6.3mm_D2.5mm_P7.62mm_Horizontal, symbol Device:R_US
- added D18, D19, D20, D24, D25, D26, D30, D31, D32: LED, LED_THT:LED_D3.0mm, symbol Device:LED
- added D33, D34, D35: 1N5819, digikey-footprints:DO-41, symbol dk_Diodes-Rectifiers-Single:1N5819
- added K7, K8, K9: SANYOU_SRD_Form_C, Relay_THT:Relay_SPDT_SANYOU_SRD_Series_Form_C, symbol Relay:SANYOU_SRD_Form_C
- added O7, O8, O9: PC817, Package_DIP:DIP-4_W7.62mm, symbol Isolator:PC817
- added Q7, Q8, Q9: PN2222A, digikey-footprints:TO-92-3, symbol dk_Transistors-Bipolar-BJT-Single:PN2222A
- added R19, R20, R34, R35, R36, R4, R5: 1K, Resistor_THT:R_Axial_DIN0207_L6.3mm_D2.5mm_P7.62mm_Horizontal, symbol Device:R_US
- added R37, R38, R39, R43, R44, R45, R46, R47, R48: 330, Resistor_THT:R_Axial_DIN0207_L6.3mm_D2.5mm_P7.62mm_Horizontal, symbol Device:R_US
- added R40, R41, R42: 10K, Resistor_THT:R_Axial_DIN0207_L6.3mm_D2.5mm_P7.62mm_Horizontal, symbol Device:R_US
- R21: value 330 -> 1K
- R6: renamed from R11; value 330 -> 1K
- renumbered D1 to D21, D2 to D22, D3 to D23, D4 to D27, D5 to D28, D6 to D29, R3 to R10, R8 to R11, R13 to R12, R5 to R13, R9 to R14, R14 to R15, R4 to R16, R10 to R17, R15 to R18, R17 to R22, R22 to R23, R27 to R24, R18 to R25, R23 to R26, R28 to R27, R19 to R28, R24 to R29, R29 to R30, R20 to R31, R25 to R32, R30 to R33, R2 to R7, R7 to R8, R12 to R9
Connections:
- net +12V: now also D33.K, D34.K, D35.K, K7.5, K8.5, K9.5, R43.2, R44.2, R45.2, R46.1, R47.1, R48.1
- net GND: now also Q7.1 (E), Q8.1 (E), Q9.1 (E), R19.2, R20.2, R34.2, R35.2, R36.2, R37.2, R38.2, R39.2, R4.2, R40.2, R41.2, R42.2, R5.2
- net K1: now also D18.2 (A)
- net K2: now also D19.2 (A)
- net K3: now also D20.2 (A); no longer R6.1
- net K4: now also D24.2 (A)
- net K5: now also D25.2 (A); no longer R21.1
- net K6: now also D26.2 (A)
- new net: D30.1 (K), R34.1
- new net: D24.1 (K), R19.1
- new net: O7.2, R37.1
- new net: D33.A, K7.2, Q7.3 (C), R46.2
- new net: D34.A, K8.2, Q8.3 (C), R47.2
- new net: D18.1 (K), R4.1
- new net: O8.2, R38.1
- new net: O8.3, Q8.2 (B), R41.1
- new net: O8.4, R44.1
- new net: O9.2, R39.1
- new net: D19.1 (K), R5.1
- new net: D25.1 (K), R20.1
- new net: O7.4, R43.1
- new net: D35.A, K9.2, Q9.3 (C), R48.2
- new net: O9.4, R45.1
- new net: D31.1 (K), R35.1
- new net: D26.1 (K), R21.1
- new net: D32.1 (K), R36.1
- new net: O7.3, Q7.2 (B), R40.1
- new net: O9.3, Q9.2 (B), R42.1
- new net: D20.1 (K), R6.1
- new net K7: D30.2 (A), O7.1
- new net K7_COM: K7.1
- new net K7_N_C: K7.4
- new net K7_N_O: K7.3
- new net K8: D31.2 (A), O8.1
- new net K8_COM: K8.1
- new net K8_N_C: K8.4
- new net K8_N_O: K8.3
- new net K9: D32.2 (A), O9.1
- new net K9_COM: K9.1
- new net K9_N_C: K9.4
- new net K9_N_O: K9.3
Other:
- moved on the sheet: D21, D22, D23, D27, D28, D29, K1, K2, K3, K4, K5, K6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

Commit message: PCB 90% & Corrections to diagram in the ADC section were done
Te resistors to secure a low logical level were placed, also the routing of the PCB is at the 90%
Parts:
- D21, D22, D23, D27, D28, D29, D33, D34, D35: footprint digikey-footprints:DO-41 -> Myfoodprints:D_DO-41_SOD81_P9.20mm_Horizontal
- Q1, Q2, Q3, Q4, Q5, Q6, Q7, Q8, Q9: footprint digikey-footprints:TO-92-3 -> Package_TO_SOT_THT:TO-92_Inline
Changed lines of the file:
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@@
 			)
 		)
-		(property "Footprint" "digikey-footprints:DO-41"
+		(property "Footprint" "Myfoodprints:D_DO-41_SOD81_P9.20mm_Horizontal"
 			(at 81.28 58.42 0)
 			(effects
@@
 			)
 		)
-		(property "Footprint" "digikey-footprints:DO-41"
+		(property "Footprint" "Myfoodprints:D_DO-41_SOD81_P9.20mm_Horizontal"
 			(at 218.44 160.02 0)
 			(effects
@@
 			)
 		)
-		(property "Footprint" "digikey-footprints:DO-41"
+		(property "Footprint" "Myfoodprints:D_DO-41_SOD81_P9.20mm_Horizontal"
 			(at 81.28 109.22 0)
 			(effects
@@
 			)
 		)
-		(property "Footprint" "digikey-footprints:TO-92-3"
+		(property "Footprint" "Package_TO_SOT_THT:TO-92_Inline"
 			(at 365.76 124.46 0)
 			(effects
@@
 			)
 		)
-		(property "Footprint" "digikey-footprints:TO-92-3"
+		(property "Footprint" "Package_TO_SOT_THT:TO-92_Inline"
 			(at 233.68 73.66 0)
 			(effects
@@
 			)
 		)
-		(property "Footprint" "digikey-footprints:DO-41"
+		(property "Footprint" "Myfoodprints:D_DO-41_SOD81_P9.20mm_Horizontal"
 			(at 215.9 109.22 0)
 			(effects
@@
 			)
 		)
-		(property "Footprint" "digikey-footprints:DO-41"
+		(property "Footprint" "Myfoodprints:D_DO-41_SOD81_P9.20mm_Horizontal"
 			(at 81.28 160.02 0)
 			(effects
@@
 			)
 		)
-		(property "Footprint" "digikey-footprints:TO-92-3"
+		(property "Footprint" "Package_TO_SOT_THT:TO-92_Inline"
 			(at 365.76 73.66 0)
 			(effects
@@
 			)
 		)
-		(property "Footprint" "digikey-footprints:TO-92-3"
+		(property "Footprint" "Package_TO_SOT_THT:TO-92_Inline"
 			(at 368.3 175.26 0)
 			(effects
@@
 			)
 		)
-		(property "Footprint" "digikey-footprints:TO-92-3"
+		(property "Footprint" "Package_TO_SOT_THT:TO-92_Inline"
 			(at 99.06 73.66 0)
 			(effects
@@
 			)
 		)
-		(property "Footprint" "digikey-footprints:TO-92-3"
+		(property "Footprint" "Package_TO_SOT_THT:TO-92_Inline"
 			(at 99.06 175.26 0)
 			(effects
@@
 			)
 		)
-		(property "Footprint" "digikey-footprints:DO-41"
+		(property "Footprint" "Myfoodprints:D_DO-41_SOD81_P9.20mm_Horizontal"
 			(at 350.52 160.02 0)
 			(effects
@@
 			)
 		)
-		(property "Footprint" "digikey-footprints:TO-92-3"
+		(property "Footprint" "Package_TO_SOT_THT:TO-92_Inline"
 			(at 236.22 175.26 0)
 			(effects
@@
 			)
 		)
-		(property "Footprint" "digikey-footprints:DO-41"
+		(property "Footprint" "Myfoodprints:D_DO-41_SOD81_P9.20mm_Horizontal"
 			(at 215.9 58.42 0)
 			(effects
@@
 			)
 		)
-		(property "Footprint" "digikey-footprints:DO-41"
+		(property "Footprint" "Myfoodprints:D_DO-41_SOD81_P9.20mm_Horizontal"
 			(at 347.98 58.42 0)
 			(effects
@@
 			)
 		)
-		(property "Footprint" "digikey-footprints:TO-92-3"
+		(property "Footprint" "Package_TO_SOT_THT:TO-92_Inline"
 			(at 233.68 124.46 0)
 			(effects
@@
 			)
 		)
-		(property "Footprint" "digikey-footprints:TO-92-3"
+		(property "Footprint" "Package_TO_SOT_THT:TO-92_Inline"
 			(at 99.06 124.46 0)
 			(effects
@@
 			)
 		)
-		(property "Footprint" "digikey-footprints:DO-41"
+		(property "Footprint" "Myfoodprints:D_DO-41_SOD81_P9.20mm_Horizontal"
 			(at 347.98 109.22 0)
 			(effects
