File: BATER-IA_PCB.kicad_pcb (KiCad board)
At the start: 2 copper layers, 200 x 200 mm, 124 parts, among them J1 PJ-202A, J11 Conn_01x08, J15 Conn_01x08, J17 Conn_01x08, J21 Conn_01x10, J23 Conn_01x08, J5 Conn_01x08, J8 Conn_02x18_Counter_Clockwise, K1 SANYOU_SRD_Form_C, K10 SANYOU_SRD_Form_C, K11 SANYOU_SRD_Form_C, K2 SANYOU_SRD_Form_C, K3 SANYOU_SRD_Form_C, K4 SANYOU_SRD_Form_C, K5 SANYOU_SRD_Form_C, K6 SANYOU_SRD_Form_C, K7 SANYOU_SRD_Form_C, K8 SANYOU_SRD_Form_C, K9 SANYOU_SRD_Form_C, Q1 PN2222A, Q10 PN2222A, Q11 PN2222A, Q13 AO3400A, Q2 PN2222A, Q3 PN2222A, Q4 PN2222A, Q5 PN2222A, Q6 PN2222A, Q7 PN2222A, Q8 PN2222A, Q9 PN2222A, U1 74LS245, U10 PC817, U11 PC817, U12 PC817, U13 PC817, U14 PC817, U15 PC817, U16 PC817, U17 74LS245, U2 74LS245, U3 74LS245, U4 L7805CV, U5 LD1117V33, U6 PC817, U7 PC817, U8 PC817, U9 PC817

Commit message: PCB REV 001 design
The design of the first revition of the PCB is complete.
Parts:
- removed C1: 100uF, Capacitor_THT:CP_Radial_D8.0mm_P5.00mm
- removed C2: 330nF, Capacitor_THT:C_Disc_D8.0mm_W5.0mm_P5.00mm
- removed C3, C4: 100nF, Capacitor_THT:C_Disc_D8.0mm_W5.0mm_P5.00mm
- removed C5: 10uF, Capacitor_THT:CP_Radial_D8.0mm_P5.00mm
- removed D1, D10, D11, D15, D2, D3, D4, D5, D6, D7, D8, D9: 1N5819, digikey-footprints:DO-41
- removed D12, D13, D14: 1N4001, Diode_THT:D_DO-41_SOD81_P10.16mm_Horizontal
- removed F1: 2A, Fuse:Fuseholder_Clip-5x20mm_Bel_FC-203-22_Lateral_P17.80x5.00mm_D1.17mm_Horizontal
- removed J1: PJ-202A, digikey-footprints:Barrel_Jack_5.5mmODx2.1mmID_PJ-202A
- removed J11, J15, J17, J23, J5: Conn_01x08, Connector_PinHeader_2.54mm:PinHeader_1x08_P2.54mm_Vertical
- removed J21: Conn_01x10, Connector_PinHeader_2.54mm:PinHeader_1x08_P2.54mm_Vertical
- removed J8: Conn_02x18_Counter_Clockwise, Connector_PinHeader_2.54mm:PinHeader_2x18_P2.54mm_Vertical
- removed K1, K10, K11, K2, K3, K4, K5, K6, K7, K8, K9: SANYOU_SRD_Form_C, Relay_THT:Relay_SPDT_SANYOU_SRD_Series_Form_C
- removed Q1, Q10, Q11, Q2, Q3, Q4, Q5, Q6, Q7, Q8, Q9: PN2222A, Package_TO_SOT_THT:TO-92_Inline
- removed Q13: AO3400A, Package_TO_SOT_SMD:SOT-23
- removed R1, R10, R11, R12, R14, R15, R16, R17, R19, R2, R20, R21, R22, R24, R25, R26, R27, R29, R30, R31, R32, R34, R35, R36, R37, R39, R4, R40, R41, R42, R44, R45, R46, R47, R49, R5, R50, R51, R52, R54, R55, R6, R7, R9: 330, Resistor_THT:R_Axial_DIN0207_L6.3mm_D2.5mm_P7.62mm_Horizontal
- removed R13, R18, R23, R28, R3, R33, R38, R43, R48, R53, R8: 10K, Resistor_THT:R_Axial_DIN0207_L6.3mm_D2.5mm_P7.62mm_Horizontal
- removed U1, U17, U2, U3: 74LS245, Package_DIP:DIP-20_W7.62mm_LongPads
- removed U10, U11, U12, U13, U14, U15, U16, U6, U7, U8, U9: PC817, Package_DIP:DIP-4_W7.62mm
- removed U4: L7805CV, digikey-footprints:TO-220-3
- removed U5: LD1117V33, digikey-footprints:TO-220-3
Routing:
- net 12V_DC: track 106.4 -> 0.00 mm
- net GND: track 51.9 -> 0.00 mm
- net Net-(C1-Pad1): track 20.4 -> 0.00 mm
- net +5V: track 14.8 -> 0.00 mm
- net +3.3V: track 11.6 -> 0.00 mm
- net Net-(D15-PadA): track 7.94 -> 0.00 mm
- net Net-(Q9-C): track 4.31 -> 0.00 mm
- net Net-(Q8-C): track 4.30 -> 0.00 mm
- net Net-(Q7-C): track 4.29 -> 0.00 mm
- net Net-(Q6-C): track 4.28 -> 0.00 mm
- net Net-(Q5-C): track 4.27 -> 0.00 mm
- net Net-(Q4-C): track 4.26 -> 0.00 mm
- net Net-(Q3-C): track 4.25 -> 0.00 mm
- net Net-(Q2-C): track 4.24 -> 0.00 mm
- net Net-(Q1-C): track 4.23 -> 0.00 mm
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Other:
- board outline removed

Commit message: PCB 90% & Corrections to diagram in the ADC section were done
Te resistors to secure a low logical level were placed, also the routing of the PCB is at the 90%
Parts:
- added C1: 100uF, Capacitor_THT:CP_Radial_D8.0mm_P5.00mm, F.Cu at (78.4, 212.0)
- added C2: 0.1uF, Capacitor_THT:C_Radial_D10.0mm_H12.5mm_P5.00mm, F.Cu at (212.5, 222.0)
- added C3: 100nF, Capacitor_THT:C_Disc_D8.0mm_W5.0mm_P5.00mm, F.Cu at (200.0, 210.5)
- added C4: 10uF, Capacitor_THT:CP_Radial_D8.0mm_P5.00mm, F.Cu at (207.6, 206.0)
- added C5: 1uF, Capacitor_THT:C_Radial_D10.0mm_H12.5mm_P5.00mm, F.Cu at (230.0, 220.0)
- added C6: 10uF, Capacitor_THT:C_Radial_D5.0mm_H11.0mm_P2.00mm, F.Cu at (130.1, 147.2)
- added C7: 10uF, Capacitor_THT:C_Radial_D5.0mm_H11.0mm_P2.00mm, F.Cu at (157.5, 147.5)
- added C8: 10uF, Capacitor_THT:C_Radial_D5.0mm_H11.0mm_P2.00mm, F.Cu at (186.7, 147.7)
- added CN1: CN5711, Package_SO:Texas_HSOP-8-1EP_3.9x4.9mm_P1.27mm_ThermalVias, F.Cu at (135.1, 152.9)
- added CN2: CN5711, Package_SO:Texas_HSOP-8-1EP_3.9x4.9mm_P1.27mm_ThermalVias, F.Cu at (164.2, 152.9)
- added CN3: CN5711, Package_SO:Texas_HSOP-8-1EP_3.9x4.9mm_P1.27mm_ThermalVias, F.Cu at (194.3, 152.1)
- added D1: 1N5817, Myfoodprints:D_DO-41_SOD81_P9.20mm_Horizontal, F.Cu at (75.4, 110.7)
- added D10: 3.3V, Diode_THT:D_DO-35_SOD27_P10.16mm_Horizontal, F.Cu at (97.4, 153.7)
- added D11: 1N5817, Myfoodprints:D_DO-41_SOD81_P9.20mm_Horizontal, F.Cu at (99.3, 110.7)
- added D12: 3.3V, Diode_THT:D_DO-35_SOD27_P10.16mm_Horizontal, F.Cu at (93.4, 153.7)
- added D13: 1N5817, Myfoodprints:D_DO-41_SOD81_P9.20mm_Horizontal, F.Cu at (103.9, 110.7)
- added D14: 3.3V, Diode_THT:D_DO-35_SOD27_P10.16mm_Horizontal, F.Cu at (89.4, 153.7)
- added D15: 1N5817, Myfoodprints:D_DO-41_SOD81_P9.20mm_Horizontal, F.Cu at (108.7, 110.7)
- added D16: 3.3V, Diode_THT:D_DO-35_SOD27_P10.16mm_Horizontal, F.Cu at (85.3, 153.7)
- added D17: 1N5817, Myfoodprints:D_DO-41_SOD81_P9.20mm_Horizontal, F.Cu at (84.0, 206.4)
- added D18: LED, LED_THT:LED_D3.0mm, F.Cu at (141.1, 103.3)
- added D19: LED, LED_THT:LED_D3.0mm, F.Cu at (151.7, 102.0)
- added D2: 3.3V, Diode_THT:D_DO-35_SOD27_P10.16mm_Horizontal, F.Cu at (113.6, 153.7)
- added D20: LED, LED_THT:LED_D3.0mm, F.Cu at (178.2, 112.1)
- added D21: 1N5819, Myfoodprints:D_DO-41_SOD81_P9.20mm_Horizontal, F.Cu at (128.5, 109.4)
- added D22: 1N5819, Myfoodprints:D_DO-41_SOD81_P9.20mm_Horizontal, F.Cu at (155.7, 102.2)
- added D23: 1N5819, Myfoodprints:D_DO-41_SOD81_P9.20mm_Horizontal, F.Cu at (177.7, 127.5)
- added D24: LED, LED_THT:LED_D3.0mm, F.Cu at (208.8, 143.6)
- added D25: LED, LED_THT:LED_D3.0mm, F.Cu at (223.7, 135.8)
- added D26: LED, LED_THT:LED_D3.0mm, F.Cu at (242.8, 127.8)
- added D27: 1N5819, Myfoodprints:D_DO-41_SOD81_P9.20mm_Horizontal, F.Cu at (199.5, 96.1)
- added D28: 1N5819, Myfoodprints:D_DO-41_SOD81_P9.20mm_Horizontal, F.Cu at (224.3, 103.4)
- added D29: 1N5819, Myfoodprints:D_DO-41_SOD81_P9.20mm_Horizontal, F.Cu at (247.2, 120.0)
- added D3: 1N5817, Myfoodprints:D_DO-41_SOD81_P9.20mm_Horizontal, F.Cu at (80.0, 110.7)
- added D30: LED, LED_THT:LED_D3.0mm, F.Cu at (227.7, 168.1)
- added D31: LED, LED_THT:LED_D3.0mm, F.Cu at (233.2, 182.0)
- added D32: LED, LED_THT:LED_D3.0mm, F.Cu at (240.4, 214.4)
- added D33: 1N5819, Myfoodprints:D_DO-41_SOD81_P9.20mm_Horizontal, F.Cu at (245.6, 155.1)
- added D34: 1N5819, Myfoodprints:D_DO-41_SOD81_P9.20mm_Horizontal, F.Cu at (245.8, 198.4)
- added D35: 1N5819, Myfoodprints:D_DO-41_SOD81_P9.20mm_Horizontal, F.Cu at (258.7, 226.3)
- added D36: LED, LED_THT:LED_D3.0mm, F.Cu at (191.0, 206.5)
- added D37: 1N4007, Diode_THT:D_DO-41_SOD81_P10.16mm_Horizontal, F.Cu at (214.9, 197.5)
- added D38: 5V, Diode_THT:D_DO-35_SOD27_P10.16mm_Horizontal, F.Cu at (214.9, 191.5)
- added D39: LED, LED_THT:LED_D3.0mm, F.Cu at (217.4, 184.6)
- added D4: 3.3V, Diode_THT:D_DO-35_SOD27_P10.16mm_Horizontal, F.Cu at (109.6, 153.7)
- added D40: 1N5819, Myfoodprints:D_DO-41_SOD81_P9.20mm_Horizontal, F.Cu at (140.7, 137.6)
- added D41: 5V, Diode_THT:D_DO-35_SOD27_P10.16mm_Horizontal, F.Cu at (73.4, 190.8)
- added D42: 1N5819, Myfoodprints:D_DO-41_SOD81_P9.20mm_Horizontal, F.Cu at (168.7, 137.6)
- added D43: 1N5819, Myfoodprints:D_DO-41_SOD81_P9.20mm_Horizontal, F.Cu at (196.9, 139.1)
- added D5: 1N5817, Myfoodprints:D_DO-41_SOD81_P9.20mm_Horizontal, F.Cu at (84.8, 110.7)
- added D6: 3.3V, Diode_THT:D_DO-35_SOD27_P10.16mm_Horizontal, F.Cu at (105.5, 153.7)
- added D7: 1N5817, Myfoodprints:D_DO-41_SOD81_P9.20mm_Horizontal, F.Cu at (89.7, 110.7)
- added D8: 3.3V, Diode_THT:D_DO-35_SOD27_P10.16mm_Horizontal, F.Cu at (101.5, 153.7)
- added D9: 1N5817, Myfoodprints:D_DO-41_SOD81_P9.20mm_Horizontal, F.Cu at (94.5, 110.7)
- added DC-DC1: XL6019, CHN_DCDC:XL6019 MODULE, F.Cu at (113.5, 194.0)
- added DC-DC2: XL6019, CHN_DCDC:XL6019 MODULE, F.Cu at (143.0, 194.0)
- added DC-DC3: XL6019, CHN_DCDC:XL6019 MODULE, F.Cu at (172.5, 194.0)
- added F1: 2A, Fuse:Fuseholder_Clip-5x20mm_Bel_FC-203-22_Lateral_P17.80x5.00mm_D1.17mm_Horizontal, F.Cu at (91.5, 224.0)
- added H1: MountingHole, MountingHole:MountingHole_2.2mm_M2_DIN965_Pad_TopBottom, F.Cu at (74.0, 34.0)
- added H2: MountingHole, MountingHole:MountingHole_2.2mm_M2_DIN965_Pad_TopBottom, F.Cu at (266.0, 34.0)
- added H3: MountingHole, MountingHole:MountingHole_2.2mm_M2_DIN965_Pad_TopBottom, F.Cu at (266.0, 226.0)
- added H4: MountingHole, MountingHole:MountingHole_2.2mm_M2_DIN965_Pad_TopBottom, F.Cu at (110.0, 223.0)
- added INA1: INA226, Universal_Modules:INA226 Module, F.Cu at (86.9, 191.5)
- added J1: MCU_ADC_IN, Connector_PinHeader_2.54mm:PinHeader_1x08_P2.54mm_Vertical, F.Cu at (85.6, 126.2)
- added J10: PWM CH4, Connector_PinHeader_2.54mm:PinHeader_1x03_P2.54mm_Vertical, F.Cu at (206.0, 38.8)
- added J11: PWM CH5, Connector_PinHeader_2.54mm:PinHeader_1x03_P2.54mm_Vertical, F.Cu at (216.1, 38.8)
- added J12: PWM CH6, Connector_PinHeader_2.54mm:PinHeader_1x03_P2.54mm_Vertical, F.Cu at (226.1, 38.8)
- added J13: PWM GP CH1, Connector_PinHeader_2.54mm:PinHeader_1x03_P2.54mm_Vertical, F.Cu at (246.8, 38.8)
- added J14: PWM GP CH2, Connector_PinHeader_2.54mm:PinHeader_1x03_P2.54mm_Vertical, F.Cu at (241.7, 38.8)
- added J15: PWM GP CH3, Connector_PinHeader_2.54mm:PinHeader_1x03_P2.54mm_Vertical, F.Cu at (236.8, 38.8)
- added J16: STP_MOTOR_1, digikey-footprints:PinHeader_1x5_P2.5mm_Drill1.1mm, F.Cu at (264.9, 49.7)
- added J17: STP_MOTOR_2, digikey-footprints:PinHeader_1x5_P2.5mm_Drill1.1mm, F.Cu at (264.9, 66.2)
- added J18: STP_MOTOR_3, digikey-footprints:PinHeader_1x5_P2.5mm_Drill1.1mm, F.Cu at (264.9, 82.7)
- added J19: CELL 1, digikey-footprints:PinHeader_1x2_P2.5mm_Drill1.1mm, F.Cu at (242.8, 92.3)
- added J2: MCU_I2C_1, Connector_PinHeader_2.54mm:PinHeader_1x03_P2.54mm_Vertical, F.Cu at (74.7, 186.4)
- added J20: CELL 2, digikey-footprints:PinHeader_1x2_P2.5mm_Drill1.1mm, F.Cu at (253.8, 92.3)
- added J21: CELL 3, digikey-footprints:PinHeader_1x2_P2.5mm_Drill1.1mm, F.Cu at (264.9, 92.3)
- added J22: LIN ACT 1, digikey-footprints:PinHeader_1x2_P2.5mm_Drill1.1mm, F.Cu at (252.3, 143.3)
- added J23: LIN ACT 2, digikey-footprints:PinHeader_1x2_P2.5mm_Drill1.1mm, F.Cu at (252.2, 173.3)
- added J24: LIN ACT 3, digikey-footprints:PinHeader_1x2_P2.5mm_Drill1.1mm, F.Cu at (252.0, 203.5)
- added J25: CN5711_1, Connector_PinSocket_2.54mm:PinSocket_1x04_P2.54mm_Vertical, F.Cu at (134.6, 142.9)
- added J26: CN5711_2, Connector_PinSocket_2.54mm:PinSocket_1x04_P2.54mm_Vertical, F.Cu at (161.9, 142.9)
- added J27: CN5711_3, Connector_PinSocket_2.54mm:PinSocket_1x04_P2.54mm_Vertical, F.Cu at (192.0, 143.9)
- added J28: GP_ADC, Connector_PinHeader_2.54mm:PinHeader_1x04_P2.54mm_Vertical, F.Cu at (119.9, 158.8)
- added J3: MCU_PWM_INPUT, Connector_PinHeader_2.54mm:PinHeader_1x12_P2.54mm_Vertical, F.Cu at (78.2, 55.1)
- added J4: MCU_GPIOS_NPUT, Connector_PinHeader_2.54mm:PinHeader_2x17_P2.54mm_Vertical, F.Cu at (87.4, 39.9)
- added J5: GPIOS, Connector_PinHeader_2.54mm:PinHeader_1x08_P2.54mm_Vertical, F.Cu at (149.3, 38.6)
- added J6: PJ-202A, Connector_BarrelJack:BarrelJack_Horizontal, F.Cu at (83.8, 222.7)
- added J7: PWM CH1, Connector_PinHeader_2.54mm:PinHeader_1x03_P2.54mm_Vertical, F.Cu at (175.8, 38.8)
- added J8: PWM CH2, Connector_PinHeader_2.54mm:PinHeader_1x03_P2.54mm_Vertical, F.Cu at (185.9, 38.8)
- added J9: PWM CH3, Connector_PinHeader_2.54mm:PinHeader_1x03_P2.54mm_Vertical, F.Cu at (195.9, 38.8)
- added K1: SANYOU_SRD_Form_C, Relay_THT:Relay_SPDT_SANYOU_SRD_Series_Form_C, F.Cu at (134.0, 115.4)
- added K2: SANYOU_SRD_Form_C, Relay_THT:Relay_SPDT_SANYOU_SRD_Series_Form_C, F.Cu at (162.0, 115.4)
- added K3: SANYOU_SRD_Form_C, Relay_THT:Relay_SPDT_SANYOU_SRD_Series_Form_C, F.Cu at (190.1, 115.4)
- added K4: SANYOU_SRD_Form_C, Relay_THT:Relay_SPDT_SANYOU_SRD_Series_Form_C, F.Cu at (214.5, 103.4)
- added K5: SANYOU_SRD_Form_C, Relay_THT:Relay_SPDT_SANYOU_SRD_Series_Form_C, F.Cu at (236.0, 103.4)
- added K6: SANYOU_SRD_Form_C, Relay_THT:Relay_SPDT_SANYOU_SRD_Series_Form_C, F.Cu at (257.5, 103.4)
- added K7: SANYOU_SRD_Form_C, Relay_THT:Relay_SPDT_SANYOU_SRD_Series_Form_C, F.Cu at (250.7, 158.0)
- added K8: SANYOU_SRD_Form_C, Relay_THT:Relay_SPDT_SANYOU_SRD_Series_Form_C, F.Cu at (250.5, 188.1)
- added K9: SANYOU_SRD_Form_C, Relay_THT:Relay_SPDT_SANYOU_SRD_Series_Form_C, F.Cu at (250.5, 215.0)
- added O1: PC817, Package_DIP:DIP-4_W7.62mm, F.Cu at (131.1, 106.8)
- added O2: PC817, Package_DIP:DIP-4_W7.62mm, F.Cu at (161.3, 106.9)
- added O3: PC817, Package_DIP:DIP-4_W7.62mm, F.Cu at (189.3, 106.8)
- added O4: PC817, Package_DIP:DIP-4_W7.62mm, F.Cu at (207.1, 131.5)
- added O5: PC817, Package_DIP:DIP-4_W7.62mm, F.Cu at (229.1, 131.4)
- added O6: PC817, Package_DIP:DIP-4_W7.62mm, F.Cu at (247.1, 126.9)
- added O7: PC817, Package_DIP:DIP-4_W7.62mm, F.Cu at (231.2, 165.9)
- added O8: PC817, Package_DIP:DIP-4_W7.62mm, F.Cu at (231.2, 185.9)
- added O9: PC817, Package_DIP:DIP-4_W7.62mm, F.Cu at (229.1, 204.9)
- added Q1: PN2222A, Package_TO_SOT_THT:TO-92_Inline, F.Cu at (124.8, 102.6)
- added Q10: ULN2003D1013TR, digikey-footprints:SOIC-16_W3.90mm, B.Cu at (257.9, 44.6)
- added Q11: ULN2003ADR, digikey-footprints:SOIC-16_W3.90mm, B.Cu at (257.9, 69.8)
- added Q2: PN2222A, Package_TO_SOT_THT:TO-92_Inline, F.Cu at (163.8, 101.6)
- added Q3: PN2222A, Package_TO_SOT_THT:TO-92_Inline, F.Cu at (182.5, 109.0)
- added Q4: PN2222A, Package_TO_SOT_THT:TO-92_Inline, F.Cu at (217.5, 127.9)
- added Q5: PN2222A, Package_TO_SOT_THT:TO-92_Inline, F.Cu at (227.0, 126.8)
- added Q6: PN2222A, Package_TO_SOT_THT:TO-92_Inline, F.Cu at (259.4, 128.0)
- added Q7: PN2222A, Package_TO_SOT_THT:TO-92_Inline, F.Cu at (242.8, 172.1)
- added Q8: PN2222A, Package_TO_SOT_THT:TO-92_Inline, F.Cu at (259.5, 172.0)
- added Q9: PN2222A, Package_TO_SOT_THT:TO-92_Inline, F.Cu at (244.4, 207.9)
- added R1: 5.1, Resistor_THT:R_Axial_DIN0614_L14.3mm_D5.7mm_P15.24mm_Horizontal, F.Cu at (191.1, 182.3)
- added R10: 10K, Resistor_THT:R_Axial_DIN0207_L6.3mm_D2.5mm_P7.62mm_Horizontal, F.Cu at (151.3, 115.0)
- added R11: 10K, Resistor_THT:R_Axial_DIN0207_L6.3mm_D2.5mm_P7.62mm_Horizontal, F.Cu at (171.5, 125.0)
- added R12: 10K, Resistor_THT:R_Axial_DIN0207_L6.3mm_D2.5mm_P7.62mm_Horizontal, F.Cu at (195.2, 99.5)
- added R13: 330, Resistor_THT:R_Axial_DIN0207_L6.3mm_D2.5mm_P7.62mm_Horizontal, F.Cu at (146.6, 107.4)
- added R14: 330, Resistor_THT:R_Axial_DIN0207_L6.3mm_D2.5mm_P7.62mm_Horizontal, F.Cu at (173.2, 105.1)
- added R15: 330, Resistor_THT:R_Axial_DIN0207_L6.3mm_D2.5mm_P7.62mm_Horizontal, F.Cu at (199.6, 98.8)
- added R16: 330, Resistor_THT:R_Axial_DIN0207_L6.3mm_D2.5mm_P7.62mm_Horizontal, F.Cu at (146.6, 117.4)
- added R17: 330, Resistor_THT:R_Axial_DIN0207_L6.3mm_D2.5mm_P7.62mm_Horizontal, F.Cu at (171.6, 114.9)
- added R18: 330, Resistor_THT:R_Axial_DIN0207_L6.3mm_D2.5mm_P7.62mm_Horizontal, F.Cu at (199.6, 116.3)
- added R19: 1K, Resistor_THT:R_Axial_DIN0207_L6.3mm_D2.5mm_P7.62mm_Horizontal, F.Cu at (213.5, 142.1)
- added R2: 5.1, Resistor_THT:R_Axial_DIN0614_L14.3mm_D5.7mm_P15.24mm_Horizontal, F.Cu at (199.7, 182.3)
- added R20: 1K, Resistor_THT:R_Axial_DIN0207_L6.3mm_D2.5mm_P7.62mm_Horizontal, F.Cu at (224.5, 138.1)
- added R21: 1K, Resistor_THT:R_Axial_DIN0207_L6.3mm_D2.5mm_P7.62mm_Horizontal, F.Cu at (243.5, 130.3)
- added R22: 330, Resistor_THT:R_Axial_DIN0207_L6.3mm_D2.5mm_P7.62mm_Horizontal, F.Cu at (207.1, 138.4)
- added R23: 330, Resistor_THT:R_Axial_DIN0207_L6.3mm_D2.5mm_P7.62mm_Horizontal, F.Cu at (229.1, 138.1)
- added R24: 330, Resistor_THT:R_Axial_DIN0207_L6.3mm_D2.5mm_P7.62mm_Horizontal, F.Cu at (254.7, 137.5)
- added R25: 10K, Resistor_THT:R_Axial_DIN0207_L6.3mm_D2.5mm_P7.62mm_Horizontal, F.Cu at (218.5, 138.1)
- added R26: 10K, Resistor_THT:R_Axial_DIN0207_L6.3mm_D2.5mm_P7.62mm_Horizontal, F.Cu at (234.5, 138.0)
- added R27: 10K, Resistor_THT:R_Axial_DIN0207_L6.3mm_D2.5mm_P7.62mm_Horizontal, F.Cu at (257.5, 132.3)
- added R28: 330, Resistor_THT:R_Axial_DIN0207_L6.3mm_D2.5mm_P7.62mm_Horizontal, F.Cu at (204.5, 127.1)
- added R29: 330, Resistor_THT:R_Axial_DIN0207_L6.3mm_D2.5mm_P7.62mm_Horizontal, F.Cu at (239.4, 138.1)
- added R3: 5.1, Resistor_THT:R_Axial_DIN0614_L14.3mm_D5.7mm_P15.24mm_Horizontal, F.Cu at (208.3, 182.3)
- added R30: 330, Resistor_THT:R_Axial_DIN0207_L6.3mm_D2.5mm_P7.62mm_Horizontal, F.Cu at (262.6, 132.3)
- added R31: 330, Resistor_THT:R_Axial_DIN0207_L6.3mm_D2.5mm_P7.62mm_Horizontal, F.Cu at (207.3, 126.7)
- added R32: 330, Resistor_THT:R_Axial_DIN0207_L6.3mm_D2.5mm_P7.62mm_Horizontal, F.Cu at (221.3, 100.1)
- added R33: 330, Resistor_THT:R_Axial_DIN0207_L6.3mm_D2.5mm_P7.62mm_Horizontal, F.Cu at (246.9, 107.0)
- added R34: 1K, Resistor_THT:R_Axial_DIN0207_L6.3mm_D2.5mm_P7.62mm_Horizontal, F.Cu at (227.7, 170.3)
- added R35: 1K, Resistor_THT:R_Axial_DIN0207_L6.3mm_D2.5mm_P7.62mm_Horizontal, F.Cu at (227.9, 184.8)
- added R36: 1K, Resistor_THT:R_Axial_DIN0207_L6.3mm_D2.5mm_P7.62mm_Horizontal, F.Cu at (246.3, 218.9)
- added R37: 330, Resistor_THT:R_Axial_DIN0207_L6.3mm_D2.5mm_P7.62mm_Horizontal, F.Cu at (231.7, 175.2)
- added R38: 330, Resistor_THT:R_Axial_DIN0207_L6.3mm_D2.5mm_P7.62mm_Horizontal, F.Cu at (231.7, 192.0)
- added R39: 330, Resistor_THT:R_Axial_DIN0207_L6.3mm_D2.5mm_P7.62mm_Horizontal, F.Cu at (243.2, 221.9)
- added R4: 1K, Resistor_THT:R_Axial_DIN0207_L6.3mm_D2.5mm_P7.62mm_Horizontal, F.Cu at (137.9, 103.4)
- added R40: 10K, Resistor_THT:R_Axial_DIN0207_L6.3mm_D2.5mm_P7.62mm_Horizontal, F.Cu at (231.2, 171.6)
- added R41: 10K, Resistor_THT:R_Axial_DIN0207_L6.3mm_D2.5mm_P7.62mm_Horizontal, F.Cu at (242.1, 184.9)
- added R42: 10K, Resistor_THT:R_Axial_DIN0207_L6.3mm_D2.5mm_P7.62mm_Horizontal, F.Cu at (236.6, 210.6)
- added R43: 330, Resistor_THT:R_Axial_DIN0207_L6.3mm_D2.5mm_P7.62mm_Horizontal, F.Cu at (238.5, 152.2)
- added R44: 330, Resistor_THT:R_Axial_DIN0207_L6.3mm_D2.5mm_P7.62mm_Horizontal, F.Cu at (240.3, 178.3)
- added R45: 330, Resistor_THT:R_Axial_DIN0207_L6.3mm_D2.5mm_P7.62mm_Horizontal, F.Cu at (256.3, 201.3)
- added R46: 330, Resistor_THT:R_Axial_DIN0207_L6.3mm_D2.5mm_P7.62mm_Horizontal, F.Cu at (242.3, 154.8)
- added R47: 330, Resistor_THT:R_Axial_DIN0207_L6.3mm_D2.5mm_P7.62mm_Horizontal, F.Cu at (246.8, 185.0)
- added R48: 330, Resistor_THT:R_Axial_DIN0207_L6.3mm_D2.5mm_P7.62mm_Horizontal, F.Cu at (263.9, 204.4)
- added R49: 270, Resistor_THT:R_Axial_DIN0411_L9.9mm_D3.6mm_P12.70mm_Horizontal, F.Cu at (242.2, 227.5)
- added R5: 1K, Resistor_THT:R_Axial_DIN0207_L6.3mm_D2.5mm_P7.62mm_Horizontal, F.Cu at (150.5, 99.2)
- added R50: 1K, Resistor_THT:R_Axial_DIN0204_L3.6mm_D1.6mm_P5.08mm_Horizontal, F.Cu at (191.0, 202.2)
- added R51: 1K, Resistor_THT:R_Axial_DIN0204_L3.6mm_D1.6mm_P5.08mm_Horizontal, F.Cu at (219.9, 184.6)
- added R52: 10K, Resistor_THT:R_Axial_DIN0207_L6.3mm_D2.5mm_P7.62mm_Horizontal, F.Cu at (149.4, 148.8)
- added R53: 10K, Resistor_THT:R_Axial_DIN0207_L6.3mm_D2.5mm_P7.62mm_Horizontal, F.Cu at (177.5, 147.0)
- added R54: 10K, Resistor_THT:R_Axial_DIN0207_L6.3mm_D2.5mm_P7.62mm_Horizontal, F.Cu at (208.0, 147.7)
- added R6: 1K, Resistor_THT:R_Axial_DIN0207_L6.3mm_D2.5mm_P7.62mm_Horizontal, F.Cu at (178.2, 109.7)
- added R67: 10K, Resistor_THT:R_Axial_DIN0207_L6.3mm_D2.5mm_P7.62mm_Horizontal, F.Cu at (79.8, 125.9)
- added R68: 10K, Resistor_THT:R_Axial_DIN0207_L6.3mm_D2.5mm_P7.62mm_Horizontal, F.Cu at (79.8, 130.5)
- added R69: 10K, Resistor_THT:R_Axial_DIN0207_L6.3mm_D2.5mm_P7.62mm_Horizontal, F.Cu at (79.8, 135.1)
- added R7: 330, Resistor_THT:R_Axial_DIN0207_L6.3mm_D2.5mm_P7.62mm_Horizontal, F.Cu at (123.7, 114.2)
- added R70: 10K, Resistor_THT:R_Axial_DIN0207_L6.3mm_D2.5mm_P7.62mm_Horizontal, F.Cu at (79.8, 139.7)
- added R71: 10K, Resistor_THT:R_Axial_DIN0207_L6.3mm_D2.5mm_P7.62mm_Horizontal, F.Cu at (79.8, 144.3)
- added R72: 10K, Resistor_THT:R_Axial_DIN0207_L6.3mm_D2.5mm_P7.62mm_Horizontal, F.Cu at (79.8, 149.0)
- added R73: 10K, Resistor_THT:R_Axial_DIN0207_L6.3mm_D2.5mm_P7.62mm_Horizontal, F.Cu at (79.8, 153.6)
- added R74: 10K, Resistor_THT:R_Axial_DIN0207_L6.3mm_D2.5mm_P7.62mm_Horizontal, F.Cu at (79.8, 158.2)
- added R8: 330, Resistor_THT:R_Axial_DIN0207_L6.3mm_D2.5mm_P7.62mm_Horizontal, F.Cu at (160.8, 104.2)
- added R9: 330, Resistor_THT:R_Axial_DIN0207_L6.3mm_D2.5mm_P7.62mm_Horizontal, F.Cu at (185.4, 99.5)
- added R_POT1: 2K, Potentiometer_THT:Potentiometer_Bourns_3296W_Vertical, F.Cu at (222.5, 215.0)
- added R_POT2: 2K, Potentiometer_THT:Potentiometer_Bourns_3296W_Vertical, F.Cu at (222.5, 206.0)
- added R_POT3: 2K, Potentiometer_THT:Potentiometer_Bourns_3296W_Vertical, F.Cu at (143.3, 154.9)
- added R_POT4: 2K, Potentiometer_THT:Potentiometer_Bourns_3296W_Vertical, F.Cu at (171.7, 153.1)
- added R_POT5: 2K, Potentiometer_THT:Potentiometer_Bourns_3296W_Vertical, F.Cu at (202.2, 154.1)
- added SHORT_1: 0, Myfoodprints:Short_5.08mm_Drill1.3mm, F.Cu at (140.5, 163.3)
- added SHORT_2: 0, Myfoodprints:Short_5.08mm_Drill1.3mm, F.Cu at (145.5, 163.3)
- added U1: 74LS245, Package_DIP:DIP-20_W7.62mm_LongPads, F.Cu at (85.3, 52.3)
- added U2: 74LS245, Package_DIP:DIP-20_W7.62mm_LongPads, F.Cu at (85.3, 81.8)
- added U3: 74LS245, Package_DIP:DIP-20_W7.62mm_LongPads, F.Cu at (106.9, 81.8)
- added U4: 74LS245, Package_DIP:DIP-20_W7.62mm_LongPads, F.Cu at (106.4, 52.3)
- added U5: 74LS245, Package_DIP:DIP-20_W7.62mm_LongPads, F.Cu at (131.1, 52.3)
- added U6: LD1117V33, Package_TO_SOT_THT:TO-220-3_Vertical, F.Cu at (199.0, 224.0)
- added U7: LM338T, Package_TO_SOT_THT:TO-220-3_Vertical, F.Cu at (225.0, 224.0)
Routing:
- net GND: track 0.00 -> 2201.9 mm, vias 0 -> 5
- net +12V: track 0.00 -> 885.6 mm
- net +5V: track 0.00 -> 371.9 mm, vias 0 -> 2
- net +3.3V: track 0.00 -> 281.6 mm, vias 0 -> 1
- net PWM_5V_GP_2: track 0.00 -> 241.7 mm, vias 0 -> 2
- net PWM_5V_GP_1: track 0.00 -> 221.0 mm, vias 0 -> 4
- net PWM_SERVO_6: track 0.00 -> 184.2 mm, vias 0 -> 5
- net D33_5V: track 0.00 -> 179.5 mm, vias 0 -> 6
- net D32_5V: track 0.00 -> 177.1 mm, vias 0 -> 6
- net D37_5V: track 0.00 -> 174.0 mm, vias 0 -> 2
- net D36_5V: track 0.00 -> 173.8 mm, vias 0 -> 2
- net D31_5V: track 0.00 -> 169.2 mm, vias 0 -> 4
- net D34_5V: track 0.00 -> 167.6 mm, vias 0 -> 3
- net D35_5V: track 0.00 -> 166.4 mm, vias 0 -> 2
- net PWM_SERVO_5: track 0.00 -> 162.6 mm, vias 0 -> 5
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Other:
- board outline added: 200 x 200 mm

Commit message: Rev 01 has been finished
gerber files , drill files and map drill has been generated
Parts:
- moved J21 3.36 mm to (261.6, 92.9)
- moved J6 0.51 mm to (84.2, 222.9)
Routing:
- net D26_5V: track 6.14 -> 313.1 mm, vias 0 -> 3
- net D30_5V: track 13.2 -> 277.7 mm, vias 0 -> 6
- net D27_5V: track 5.03 -> 230.7 mm
- net +5V: track 371.9 -> 591.8 mm, vias 2 -> 4
- net D29_5V: track 4.19 -> 197.4 mm, vias 0 -> 5
- net ADC_CH5: track 55.1 -> 228.7 mm
- net ADC_CH4: track 52.7 -> 221.2 mm
- net D28_5V: track 3.63 -> 167.6 mm, vias 0 -> 6
- net D25_5V: track 13.3 -> 174.1 mm, vias 0 -> 2
- net ADC_CH3: track 50.3 -> 198.3 mm
- net GND: track 2201.9 -> 2345.6 mm
- net /BUFFER LEVEL SHIFTER/PWM3_5V: track 28.4 -> 165.5 mm, vias 0 -> 6
- net /BUFFER LEVEL SHIFTER/PWM4_5V: track 28.5 -> 163.0 mm, vias 0 -> 5
- net D24_5V: track 16.1 -> 140.6 mm, vias 2 -> 3
- net CELL_2: track 22.5 -> 140.4 mm, vias 0 -> 1
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- added copper zone on B.Cu, net GND
- added copper zone on F.Cu, net GND
